File: placa_iot/_autosave-MCU.kicad_sch (KiCad schematic)
At the start: 31 parts, among them J1 22-28-4144, J2 22-28-4144, SW1 RST/EN, SW2 BOOT, U3 ESP32-S3, U4 PRO-OB-536, Y1 40MHz

Commit message: RF
Parts:
- C15, C16, C18, C20: now not fitted
Changed lines of the file:
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@@
 		(on_board yes)
 		(in_pos_files yes)
-		(dnp no)
+		(dnp yes)
 		(fields_autoplaced yes)
 		(property "Reference" "C20"
@@
 		(on_board yes)
 		(in_pos_files yes)
-		(dnp no)
+		(dnp yes)
 		(fields_autoplaced yes)
 		(property "Reference" "C18"
@@
 		(on_board yes)
 		(in_pos_files yes)
-		(dnp no)
+		(dnp yes)
 		(fields_autoplaced yes)
 		(property "Reference" "C15"
@@
 		(on_board yes)
 		(in_pos_files yes)
-		(dnp no)
+		(dnp yes)
 		(fields_autoplaced yes)
 		(property "Reference" "C16"

Commit message: SQUEMATIC FINISH
Parts:
- added D6: LED, LED_SMD:LED_0402_1005Metric, symbol Device:LED
- added R24: 1 KOhm, Resistor_SMD:R_0402_1005Metric, symbol Device:R
Connections:
- net IO2 is gone; now on net IO1: U3.6 (GPIO1)
- net IO48 is gone; now on net IO36: J2.8 (Pin_8), U3.36 (SPICLK_N)
- net GND: now also D6.1 (K)
- net IO47: now also R24.2
- net IO19 renamed D+
- net IO20 renamed D-
- new net: D6.2 (A), R24.1
