File: placa_iot/MCU.kicad_sch (KiCad schematic)
At the start: 0 parts

Commit message: microcontrolador en proceso
Parts:
- added C10, C6, C9: 1uF, Capacitor_SMD:C_0402_1005Metric, symbol Device:C
- added C11, C12: 10uF, Capacitor_SMD:C_0402_1005Metric, symbol Device:C
- added C13: 12uF, Capacitor_SMD:C_0402_1005Metric, symbol Device:C
- added C14: 9uF, Capacitor_SMD:C_0402_1005Metric, symbol Device:C
- added C15, C16, C17, C18, C19, C20: NC, Capacitor_SMD:C_0402_1005Metric, symbol Device:C
- added C21, C8: 100nF, Capacitor_SMD:C_0402_1005Metric, symbol Device:C
- added C7: 10nF, Capacitor_SMD:C_0402_1005Metric, symbol Device:C
- added L1: 2nH, Inductor_SMD:L_0402_1005Metric, symbol Device:L
- added L2: 22nH, Inductor_SMD:L_0402_1005Metric, symbol Device:L
- added R4: NC, Resistor_SMD:R_0402_1005Metric, symbol Device:R
- added R5: 499 Ohm, Resistor_SMD:R_0402_1005Metric, symbol Device:R
- added U3: ESP32-S3, ic_control:QFN-56-1EP_7x7mm_P0.4mm_EP4x4mm, symbol ic_control:ESP32-S3
- added U4: PRO-OB-536, antennas:ANTENNA_PIFA_3D_2.4GHZ, symbol antenas:ANTENNA_PIFA_3D_2.4GHZ
- added Y1: 40MHz, Crystal:Crystal_SMD_3225-4Pin_3.2x2.5mm, symbol Device:Crystal_GND24
Connections:
- new net: C19.2, C20.1, U4.2 (FEED)
- new net: R5.2, U3.49 (U0TXD)
- new net: C15.1, C17.1, U3.1 (LNA_IN)
- new net: C12.1, L1.2, U3.2 (VDD3P3), U3.3 (VDD3P3)
- new net: C14.1, U3.53 (XTAL_N), Y1.3
- new net: L2.2, U3.54 (XTAL_P)
- new net: C16.1, C17.2, C18.1, C19.1
- new net: C13.1, L2.1, Y1.1
- new net +3V3: C10.1, C11.1, C21.1, C6.1, C7.1, C8.1, C9.1, L1.1, R4.2, U3.20 (VDD3P3_RTC), U3.46 (VDD3P3_CPU), U3.55 (VDDA), U3.56 (VDDA)
- new net GND: C10.2, C11.2, C12.2, C13.2, C14.2, C15.2, C16.2, C18.2, C20.2, C21.2, C6.2, C7.2, C8.2, C9.2, U3.57 (GND), U4.1 (GND), Y1.2 (G), Y1.4 (G)
- new net IO1: U3.5 (GPIO0)
- new net IO3: U3.8 (GPIO3)
- new net IO4: U3.9 (GPIO4)
- new net IO45: R4.1, U3.51 (GPIO45)
- new net IO5: U3.10 (GPIO5)
- new net IO6: U3.11 (GPIO6)
- new net IO7: U3.12 (GPIO7)
- new net IO8: U3.13 (GPIO8)
- new net IO9: U3.14 (GPIO9)
- new net LORA_TX: U3.15 (GPIO10)
- new net RST/EN: U3.16 (GPIO11), U3.17 (GPIO12), U3.18 (GPIO13), U3.19 (GPIO14), U3.23 (GPIO17), U3.24 (GPIO18), U3.25 (GPIO19/USB_D-), U3.26 (GPIO20/USB_D+), U3.27 (GPIO21), U3.4 (CHIP_PU)
- new net SDO-MISO-1O2: U3.7 (GPIO2)
- new net UOTXD: R5.1

Commit message: SQUEMATIC FINISH
Parts:
- added C22: 1uF, Capacitor_SMD:C_0402_1005Metric, symbol Device:C
- added D6: LED, LED_SMD:LED_0402_1005Metric, symbol Device:LED
- added J1, J2: 22-28-4144, connectors:CONN_THT_MV_PH_P2.54MM_P14, symbol connectors:CONN_THT_MV_PH_P2.54MM_P14
- added R24: 1 KOhm, Resistor_SMD:R_0402_1005Metric, symbol Device:R
- added R6, R7, R9: 10 KOhm, Resistor_SMD:R_0402_1005Metric, symbol Device:R
- added SW1: RST/EN, Button_Switch_SMD:SW_Push_SPST_NO_Alps_SKRK, symbol Switch:SW_Push
- added SW2: BOOT, Button_Switch_SMD:SW_Push_SPST_NO_Alps_SKRK, symbol Switch:SW_Push
- C15, C16, C18, C20: now not fitted
Connections:
- net +3V3: now also J1.1 (Pin_1), J1.3 (Pin_3), R6.1, R9.1
- net GND: now also C22.1, D6.1 (K), J1.2 (Pin_2), J1.4 (Pin_4), J2.14 (Pin_14), SW1.1, SW2.1
- net IO2: now also U3.6 (GPIO1)
- net IO45: now also J1.7 (Pin_7)
- net IO8: now also J2.9 (Pin_9)
- net RST/EN: now also J2.11 (Pin_11); no longer U3.16 (GPIO11), U3.17 (GPIO12), U3.18 (GPIO13), U3.19 (GPIO14), U3.23 (GPIO17), U3.24 (GPIO18), U3.25 (GPIO19/USB_D-), U3.26 (GPIO20/USB_D+), U3.27 (GPIO21)
- net IO21: now reaches U3.21 (XTAL_32K_P)
- net IO22: now reaches U3.22 (XTAL_32K_N)
- net IO48: now reaches U3.36 (SPICLK_N)
- net IO48: now also J2.8 (Pin_8)
- net IO47: now reaches U3.37 (SPICLK_P)
- net IO47: now also J2.7 (Pin_7), R24.2
- net IO33: now reaches U3.38 (GPIO33)
- net IO33: now also J2.6 (Pin_6)
- net IO34: now reaches U3.39 (GPIO34)
- net IO34: now also J2.5 (Pin_5)
- net IO35: now reaches U3.40 (GPIO35)
- net IO35: now also J2.4 (Pin_4)
- net IO36: now reaches U3.41 (GPIO36)
- net IO36: now also J2.2 (Pin_2)
- net IO37: now reaches U3.42 (GPIO37)
- net IO37: now also J2.1 (Pin_1)
- net IO38: now reaches U3.43 (GPIO38)
- net IO38: now also J1.13 (Pin_13)
- net IO39/MTCK: now reaches U3.44 (MTCK)
- net IO39/MTCK: now also J1.10 (Pin_10)
- net IO40/MTDO: now reaches U3.45 (MTDO)
- net IO40/MTDO: now also J1.9 (Pin_9)
- net IO41/MTDI: now reaches U3.47 (MTDI)
- net IO41/MTDI: now also J1.8 (Pin_8)
- net IO42/MTMS: now reaches U3.48 (MTMS)
- net IO42/MTMS: now also J1.5 (Pin_5)
- net U0RXD: now reaches U3.50 (U0RXD)
- net U0RXD: now also J1.11 (Pin_11)
- net IO46: now reaches U3.52 (GPIO46)
- net IO46: now also J1.6 (Pin_6)
- new net: R7.1, SW1.2
- new net: D6.2 (A), R24.1
- new net CLK-SCK-IO14: U3.19 (GPIO14)
- new net CMD-M0S1-IO11: U3.16 (GPIO11)
- new net IO0: J2.3 (Pin_3), R9.2, SW2.2
- new net IO12: J2.10 (Pin_10), U3.17 (GPIO12)
- new net IO15: J2.12 (Pin_12)
- new net IO16: J2.13 (Pin_13)
- new net IO17: U3.23 (GPIO17)
- new net IO18: U3.24 (GPIO18)
- new net IO19: U3.25 (GPIO19/USB_D-)
- new net IO20: U3.26 (GPIO20/USB_D+)
- new net ISD3-CS-IO13: U3.18 (GPIO13)
- new net LORA_RX: U3.27 (GPIO21)
- new net RST/N: C22.2, R6.2, R7.2
- new net U0TXD: J1.12 (Pin_12)
- new net VBAT: J1.14 (Pin_14)
- no-connect marks 0 -> 8
Other:
- moved on the sheet: C13, C14, L2, R4, R5, Y1

Commit message: SQUEMATIC FINISH 1
Parts:
- renumbered C11 to C10, C14 to C11, C21 to C13, C8 to C14, C17 to C16, C16 to C17, C22 to C18, C18 to C19, C19 to C20, C20 to C21, C13 to C5, C9 to C6, C6 to C7, C10 to C8, C7 to C9, D6 to D1, L2 to L1, L1 to L2, R5 to R4, R24 to R5, R4 to R6, R6 to R8
Connections:
- net IO2 is gone; now on net IO1: U3.6 (GPIO1)
- net IO48 is gone; now on net IO36: J2.8 (Pin_8), U3.36 (SPICLK_N)
- net IO19 renamed D+
- net IO20 renamed D-
Other:
- moved on the sheet: D1, R5
