File: placa_iot/RF_LORA.kicad_sch (KiCad schematic)
At the start: 0 parts

Commit message: SQUEMATIC FINISH
Parts:
- added C24, C25, C26: NC, Capacitor_SMD:C_0402_1005Metric, symbol Device:C
- added J3: 20279-001E-03, antennas:IPEX_MHF_I, symbol antenas:IPEX_MHF_I
- added R10, R11, R12, R13: 22 Ohm, Resistor_SMD:R_0402_1005Metric, symbol Device:R
- added U5: T-SX1262, ic_control:MODULE_T_SX1262, symbol ic_control:T_SX1262
Connections:
- new net: R13.1, U5.9 (BUSY)
- new net: R10.1, U5.14 (DIO3)
- new net: C25.2, C26.1, J3.1 (In)
- new net: C24.1, C25.1, U5.16 (ANT)
- new net: R11.1, U5.13 (NC)
- new net: R12.1, U5.10 (DIO1)
- new net GND: C24.2, C26.2, J3.2 (Ext), J3.3 (Ext), U5.1 (GND), U5.15 (GND), U5.8 (GND)
- new net IO3: U5.7 (MISO)
- new net IO33: R12.2
- new net IO34: R13.2
- new net IO36: U5.2 (NC)
- new net IO5: U5.5 (SCK)
- new net IO6: U5.6 (MOSI)
- new net IO7: U5.4 (NSS)
- new net IO8: U5.3 (NRESET)
- new net IO9: U5.11 (NC)
- new net LORA_RX: R10.2
- new net LORA_TX: R11.2
- new net VCC3V3: U5.12 (3.3V)

Commit message: SQUEMATIC FINISH 1
Parts:
- renumbered C24 to C22, C25 to C23, C26 to C24
Changed lines of the file:
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@@
 		(dnp no)
 		(fields_autoplaced yes)
-		(property "Reference" "#PWR049"
+		(property "Reference" "#PWR047"
 			(at 143.51 74.93 0)
 			(hide yes)
@@
 			(project "placa_iot"
 				(path "/4b6f6f4f-6102-46a5-a2d7-92c3e7324bc6/916c0938-0d3d-45c4-a866-4c96efac2fc5"
-					(reference "#PWR049")
+					(reference "#PWR047")
 					(unit 1)
 				)
@@
 		(dnp no)
 		(fields_autoplaced yes)
-		(property "Reference" "#PWR050"
+		(property "Reference" "#PWR048"
 			(at 144.78 66.04 0)
 			(hide yes)
@@
 			(project "placa_iot"
 				(path "/4b6f6f4f-6102-46a5-a2d7-92c3e7324bc6/916c0938-0d3d-45c4-a866-4c96efac2fc5"
-					(reference "#PWR050")
+					(reference "#PWR048")
 					(unit 1)
 				)
@@
 		(dnp no)
 		(fields_autoplaced yes)
-		(property "Reference" "#PWR052"
+		(property "Reference" "#PWR050"
 			(at 177.8 66.04 0)
 			(hide yes)
@@
 			(project "placa_iot"
 				(path "/4b6f6f4f-6102-46a5-a2d7-92c3e7324bc6/916c0938-0d3d-45c4-a866-4c96efac2fc5"
-					(reference "#PWR052")
+					(reference "#PWR050")
 					(unit 1)
 				)
@@
 		(dnp no)
 		(fields_autoplaced yes)
-		(property "Reference" "#PWR048"
+		(property "Reference" "#PWR046"
 			(at 95.25 109.22 0)
 			(hide yes)
@@
 			(project "placa_iot"
 				(path "/4b6f6f4f-6102-46a5-a2d7-92c3e7324bc6/916c0938-0d3d-45c4-a866-4c96efac2fc5"
-					(reference "#PWR048")
+					(reference "#PWR046")
 					(unit 1)
 				)
@@
 		(dnp no)
 		(fields_autoplaced yes)
-		(property "Reference" "#PWR051"
+		(property "Reference" "#PWR049"
 			(at 161.29 66.04 0)
 			(hide yes)
@@
 			(project "placa_iot"
 				(path "/4b6f6f4f-6102-46a5-a2d7-92c3e7324bc6/916c0938-0d3d-45c4-a866-4c96efac2fc5"
-					(reference "#PWR051")
+					(reference "#PWR049")
 					(unit 1)
 				)
@@
 		(dnp no)
 		(fields_autoplaced yes)
-		(property "Reference" "C26"
+		(property "Reference" "C24"
 			(at 165.1 53.3399 0)
 			(show_name no)
@@
 			(project "placa_iot"
 				(path "/4b6f6f4f-6102-46a5-a2d7-92c3e7324bc6/916c0938-0d3d-45c4-a866-4c96efac2fc5"
-					(reference "C26")
+					(reference "C24")
 					(unit 1)
 				)
@@
 		(dnp no)
 		(fields_autoplaced yes)
-		(property "Reference" "C24"
+		(property "Reference" "C22"
 			(at 148.59 53.3399 0)
 			(show_name no)
@@
 			(project "placa_iot"
 				(path "/4b6f6f4f-6102-46a5-a2d7-92c3e7324bc6/916c0938-0d3d-45c4-a866-4c96efac2fc5"
-					(reference "C24")
+					(reference "C22")
 					(unit 1)
 				)
@@
 		(dnp no)
 		(fields_autoplaced yes)
-		(property "Reference" "#PWR047"
+		(property "Reference" "#PWR045"
 			(at 95.25 74.93 0)
 			(hide yes)
@@
 			(project "placa_iot"
 				(path "/4b6f6f4f-6102-46a5-a2d7-92c3e7324bc6/916c0938-0d3d-45c4-a866-4c96efac2fc5"
-					(reference "#PWR047")
-					(unit 1)
-				)
-			)
-		)
-	)
-	(symbol
-		(lib_id "power:+3V3")
-		(at 74.93 92.71 0)
-		(unit 1)
-		(body_style 1)
-		(exclude_from_sim no)
-		(in_bom yes)
-		(on_board yes)
-		(in_pos_files yes)
-		(dnp no)
-		(fields_autoplaced yes)
-		(property "Reference" "#PWR045"
-			(at 74.93 96.52 0)
-			(hide yes)
-			(show_name no)
-			(do_not_autoplace no)
-			(effects
-				(font
-					(size 1.27 1.27)
-				)
-			)
-		)
-		(property "Value" "+3V3"
-			(at 74.93 87.63 0)
-			(show_name no)
-			(do_not_autoplace no)
-			(effects
-				(font
-					(size 1.27 1.27)
-				)
-			)
-		)
-		(property "Footprint" ""
-			(at 74.93 92.71 0)
-			(hide yes)
-			(show_name no)
-			(do_not_autoplace no)
-			(effects
-				(font
-					(size 1.27 1.27)
-				)
-			)
-		)
-		(property "Datasheet" ""
-			(at 74.93 92.71 0)
-			(hide yes)
-			(show_name no)
-			(do_not_autoplace no)
-			(effects
-				(font
-					(size 1.27 1.27)
-				)
-			)
-		)
-		(property "Description" "Power symbol creates a global label with name \"+3V3\""
-			(at 74.93 92.71 0)
-			(hide yes)
-			(show_name no)
-			(do_not_autoplace no)
-			(effects
-				(font
-					(size 1.27 1.27)
-				)
-			)
-		)
-		(pin "1"
-		)
-		(instances
-			(project "placa_iot"
-				(path "/4b6f6f4f-6102-46a5-a2d7-92c3e7324bc6/916c0938-0d3d-45c4-a866-4c96efac2fc5"
 					(reference "#PWR045")
 					(unit 1)
@@
 		(dnp no)
 		(fields_autoplaced yes)
-		(property "Reference" "C25"
+		(property "Reference" "C23"
 			(at 153.67 40.64 90)
 			(show_name no)
@@
 			(project "placa_iot"
 				(path "/4b6f6f4f-6102-46a5-a2d7-92c3e7324bc6/916c0938-0d3d-45c4-a866-4c96efac2fc5"
-					(reference "C25")
-					(unit 1)
-				)
+					(reference "C23")
+					(unit 1)
+				)
