File: placa_iot/_autosave-BATERIA.kicad_sch (KiCad schematic)
At the start: 24 parts, among them J4 B2B-PH-K-S(LF)(SN), J5 B2B-PH-K-S(LF)(SN), Q1 Q_PMOS, Q2 Q_PMOS, SW3 SW_SPDT, U6 CN3065

Commit message: SQUEMATIC FINISH
Connections:
- net VBUSD is gone; now on net VBUS: D3.2 (A), Q2.G
- net ID4 renamed IO4
Other:
- moved on the sheet: C23, C27, C28, C29, D2, D3, D4, D5, J4, J5, Q2, R15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

Commit message: SQUEMATIC FINISH 1
Parts:
- removed Q1: Q_PMOS, Package_TO_SOT_SMD:SOT-23, symbol Device:Q_PMOS
- added Q3: Q_PMOS, Package_TO_SOT_SMD:SOT-23, symbol Device:Q_PMOS
- SW3: footprint (none) -> Button_Switch_THT:SW_Slide_SPDT_Angled_CK_OS102011MA1Q
- renumbered C23 to C25, C27 to C26, C28 to C27, C29 to C28, D1 to D2, D2 to D3, D3 to D4, D4 to D6, R17 to R15, R15 to R16, R18 to R17, R19 to R18, R20 to R19, R21 to R20, R22 to R21, R23 to R22
Connections:
- net SOLAR_IND: now also Q2.3 (D); no longer Q2.D
- net VBAT: now also Q3.3 (D)
- net VBUS: now also Q2.1 (G), Q3.1 (G); no longer Q2.G
- net at C25.1, C26.1, D4.1 (K)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: now also Q2.2 (S); no longer Q2.S
- net at D2.1 (K), SW3.2 (B): now also Q3.2 (S)
