File: placa_iot/placa_iot.kicad_sch (KiCad schematic)
At the start: 0 parts

Commit message: SQUEMATIC FINISH 1
Other:
- added sheet USB (untitled.kicad_sch)
Changed lines of the file:
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@@
 	)
 	(sheet
-		(at 252.73 85.09)
+		(at 245.11 63.5)
 		(size 118.11 66.04)
 		(exclude_from_sim no)
@@
 		)
 		(property "Sheetname" "RF_LORA"
-			(at 252.73 84.3784 0)
+			(at 245.11 62.7884 0)
 			(show_name no)
 			(do_not_autoplace no)
@@
 		)
 		(property "Sheetfile" "RF_LORA.kicad_sch"
-			(at 252.73 151.7146 0)
+			(at 245.11 130.1246 0)
 			(show_name no)
 			(do_not_autoplace no)
@@
 				)
 			)
+		)
+	)
+	(sheet
+		(at 245.11 148.59)
+		(size 119.38 58.42)
+		(exclude_from_sim no)
+		(in_bom yes)
+		(on_board yes)
+		(dnp no)
+		(fields_autoplaced yes)
+		(stroke
+			(width 0.1524)
+			(type solid)
+		)
+		(fill
+			(color 0 0 0 0)
+		)
+		(property "Sheetname" "USB"
+			(at 245.11 147.8784 0)
+			(show_name no)
+			(do_not_autoplace no)
+			(effects
+				(font
+					(size 1.27 1.27)
+				)
+				(justify left bottom)
+			)
+		)
+		(property "Sheetfile" "untitled.kicad_sch"
+			(at 245.11 207.5946 0)
+			(show_name no)
+			(do_not_autoplace no)
+			(effects
+				(font
+					(size 1.27 1.27)
+				)
+				(justify left top)
+			)
+		)
+		(instances
+			(project "placa_iot"
+				(path "/4b6f6f4f-6102-46a5-a2d7-92c3e7324bc6"
+					(page "6")
+				)
+			)
